File: 6S_BMS_Passthrough.kicad_sch (KiCad schematic)
At the start: 42 parts, among them J1 Conn_01x08_Pin, J4 Conn_01x02_Pin, J5 Conn_01x04_Pin, J6 Conn_01x04_Pin, SW1 SW_SPST, U1 BQ76925RGER, U2 STM32L431KCUx, U3 TJA1051TK-3, U4 TCAN3404DRBRQ1

Commit message: Updated to use CAN 5V
Parts:
- removed C20, C9: 100nF, PCM_JLCPCB:C_0603, symbol PCM_JLCPCB-Capacitors:0603,100nF
- removed C21: 1uF, PCM_JLCPCB:C_0603, symbol PCM_JLCPCB-Capacitors:0603,1uF
- removed U3: TJA1051TK-3, Package_DFN_QFN:DFN-8-1EP_3x3mm_P0.65mm_EP1.55x2.4mm, symbol Interface_CAN_LIN:TJA1051TK-3
- added C2: 10uF, PCM_JLCPCB:C_0603, symbol PCM_JLCPCB-Capacitors:0603,10uF
- added C20: 1uF, PCM_JLCPCB:C_0603, symbol PCM_JLCPCB-Capacitors:0603,1uF
- added D1: BZT52C5V6, PCM_JLCPCB:D_SOD-123, symbol PCM_JLCPCB-Diodes:Zener,BZT52C5V6
- added J2: Conn_01x02_Pin, symbol Connector:Conn_01x02_Pin
- added Q1: ZXTP25040DFHTA, ZXTP:TPNP_SOT23_ZETEX_DIO, symbol 2026-03-10_01-30-46:ZXTP25040DFHTA
- added R1: 200kΩ, PCM_JLCPCB:R_0603, symbol PCM_JLCPCB-Resistors:0603,200kΩ
- added R2: 10Ω, PCM_JLCPCB:R_0603, symbol PCM_JLCPCB-Resistors:0603,10Ω
- added U3: TVS2700DRV, Package_SON:WSON-6-1EP_2x2mm_P0.65mm_EP1x1.6mm, symbol Power_Protection:TVS2700DRV
Connections:
- net +BATT: now also R16.1, R16.2, U1.24 (BAT), C20.1, D1.1, J2.1 (Pin_1), Q1.2, R1.1, U3.4 (IN), U3.5 (IN), U3.6 (IN)
- net CELL6P: no longer R16.1
- net GND: now also C2.2, C20.2, J2.2 (Pin_2), U3.1 (GND), U3.2 (GND), U3.3 (GND), U3.7 (GND)
- net V3P3: now also Q1.3, R2.1
- net VDD: now also C10.1, C7.2, U2.1 (VDD), U2.17 (VDD), C2.1, R2.2
- removed net BAT+: R16.2, U1.23 (VCTL), U1.24 (BAT)
- removed net PWR_5V: C10.1, C7.2, J5.1 (Pin_1), J6.4 (Pin_4), U2.1 (VDD), U2.17 (VDD)
- new net: D1.2, Q1.1, R1.2, U1.23 (VCTL)
- new net FCC_5V: J5.1 (Pin_1), J6.4 (Pin_4)
Other:
- moved on the sheet: R10, R11, R12, R13, R14, R15, R9
