File: _autosave-6S_BMS.kicad_sch (KiCad schematic)
At the start: 42 parts, among them J1 Conn_01x08_Pin, J4 Conn_01x02_Pin, J5 Conn_01x04_Pin, J6 Conn_01x04_Pin, SW1 SW_SPST, U1 BQ76925RGER, U2 STM32L431KCUx, U3 TJA1051TK-3, U4 TCAN3404DRBRQ1

Commit message: Updated to use CAN 5V
Parts:
- added R1: 10kΩ, PCM_JLCPCB:R_0603, symbol PCM_JLCPCB-Resistors:0603,10kΩ
Connections:
- net GND: now also R1.2; no longer U3.8 (S)
- new net: R1.1, U3.8 (S)
